File: pcb/bike_computer.kicad_pcb (KiCad board)
At the start: 2 copper layers, 0 parts

Commit message: Sorted main layout
Parts:
- added ANT1: SR4G008, SamacSys_Parts:SR4G008, F.Cu at (139.5, 68.5)
- added ANT2: CONUFL001-SMD, SamacSys_Parts:CONUFL001-SMD, B.Cu at (119.8, 80.8)
- added C1: 10uF, open_bike_comp:1206_0603_hand_solder, B.Cu at (139.0, 126.5)
- added C10: 0.1uF, open_bike_comp:1206_0603_hand_solder, B.Cu at (149.1, 103.3)
- added C11: 0.1uF, open_bike_comp:1206_0603_hand_solder, B.Cu at (149.1, 105.5)
- added C12: 1uF, open_bike_comp:1206_0603_hand_solder, B.Cu at (149.1, 107.7)
- added C13: 0.1uF, open_bike_comp:1206_0603_hand_solder, B.Cu at (161.5, 78.5)
- added C14: 0.1uF, open_bike_comp:1206_0603_hand_solder, B.Cu at (152.5, 78.5)
- added C15: 22pF, open_bike_comp:1206_0603_hand_solder, B.Cu at (135.2, 96.8)
- added C16: 22pF, open_bike_comp:1206_0603_hand_solder, B.Cu at (142.2, 106.8)
- added C17: 22pF, open_bike_comp:1206_0603_hand_solder, B.Cu at (142.2, 101.5)
- added C18: 0.1uF, open_bike_comp:1206_0603_hand_solder, B.Cu at (140.0, 106.7)
- added C19: 10uF, open_bike_comp:1206_0603_hand_solder, B.Cu at (128.1, 73.0)
- added C2: 10uF, open_bike_comp:1206_0603_hand_solder, B.Cu at (124.8, 130.5)
- added C20: 0.1uF, open_bike_comp:1206_0603_hand_solder, B.Cu at (130.2, 73.0)
- added C21: 0.1uF, open_bike_comp:1206_0603_hand_solder, B.Cu at (154.8, 78.5)
- added C22: 1uF, open_bike_comp:1206_0603_hand_solder, B.Cu at (117.0, 75.5)
- added C23: 33pF, open_bike_comp:1206_0603_hand_solder, B.Cu at (123.2, 73.0)
- added C24: 10pF, open_bike_comp:1206_0603_hand_solder, B.Cu at (125.5, 73.0)
- added C3: 12pF, open_bike_comp:1206_0603_hand_solder, B.Cu at (137.6, 109.6)
- added C4: 12pF, open_bike_comp:1206_0603_hand_solder, B.Cu at (137.5, 115.2)
- added C5: 10uF, open_bike_comp:1206_0603_hand_solder, B.Cu at (147.5, 129.8)
- added C6: 1uF, open_bike_comp:1206_0603_hand_solder, B.Cu at (161.6, 118.1)
- added C7: 0.1uF, open_bike_comp:1206_0603_hand_solder, B.Cu at (159.1, 118.1)
- added C8: 10uF, open_bike_comp:1206_0603_hand_solder, B.Cu at (156.1, 110.7)
- added C9: TAJC107K006SNJ, SamacSys_Parts:CAPPM6032X280N, B.Cu at (120.0, 74.5)
- added D1: 1N5819, Diode_SMD:D_SOD-123, B.Cu at (133.8, 131.2)
- added D2: 1N5819, Diode_SMD:D_SOD-123, B.Cu at (137.8, 130.0)
- added D3: ESDA6V1, SamacSys_Parts:SOT95P280X145-6N, B.Cu at (135.2, 106.5)
- added D4: 1N5819, Diode_SMD:D_SOD-123, B.Cu at (133.8, 128.8)
- added H11: Mnt_Hole_3_Top, open_bike_comp:R303000402, F.Cu at (96.5, 145.6)
- added H13: Mnt_Hole_4_Top, open_bike_comp:R303000402, F.Cu at (65.6, 145.5)
- added H7: Mnt_Hole_1_Top, open_bike_comp:R303000402, F.Cu at (56.8, 65.2)
- added H9: Mnt_Hole_2_Top, open_bike_comp:R303000402, F.Cu at (113.6, 63.3)
- added IC1: REG71050DDCR, SamacSys_Parts:SOT95P280X110-6N, B.Cu at (160.8, 112.2)
- added IC2: MPU-9250, SamacSys_Parts:QFN40P300X300X105-25N-D, B.Cu at (158.0, 78.4)
- added J1: WirelessChargeConn, Connector_PinHeader_1.27mm:PinHeader_1x02_P1.27mm_Vertical, B.Cu at (122.0, 126.5)
- added J11: 47219-2001, SamacSys_Parts:472192001, B.Cu at (155.1, 90.0)
- added J2: LiPo_Conn, Connector_PinHeader_1.27mm:PinHeader_1x02_P1.27mm_Vertical, B.Cu at (122.0, 130.8)
- added J3: Conn_01x10_TopPlate, open_bike_comp:10_smd_connector, B.Cu at (75.6, 138.2)
- added J4: SWD_header, Connector_PinHeader_2.54mm:PinHeader_1x04_P2.54mm_Vertical, F.Cu at (124.2, 135.5)
- added J5: Conn_01x10_BotPlate, Connector_PinHeader_2.54mm:PinHeader_1x10_P2.54mm_Vertical, F.Cu at (128.1, 135.5)
- added J6: 78646-3001, SamacSys_Parts:78646-3001, B.Cu at (116.8, 109.0)
- added JP1: AD0_jumper, Jumper:SolderJumper-3_P1.3mm_Open_RoundedPad1.0x1.5mm, B.Cu at (150.0, 78.5)
- added JP3: LCD_VCC_JUMPER, Jumper:SolderJumper-3_P1.3mm_Open_RoundedPad1.0x1.5mm, B.Cu at (149.2, 100.8)
- added Q1: AO3407, Package_TO_SOT_SMD:SOT-23, B.Cu at (133.8, 125.8)
- added R1: 4.7k, open_bike_comp:1206_0603_hand_solder, B.Cu at (128.5, 132.0)
- added R10: 10k, open_bike_comp:1206_0603_hand_solder, B.Cu at (145.4, 101.5)
- added R11: 10k, open_bike_comp:1206_0603_hand_solder, B.Cu at (145.4, 106.4)
- added R12: 22R, open_bike_comp:1206_0603_hand_solder, B.Cu at (133.8, 100.5)
- added R13: 22R, open_bike_comp:1206_0603_hand_solder, B.Cu at (136.5, 102.0)
- added R14: 22R, open_bike_comp:1206_0603_hand_solder, B.Cu at (140.8, 97.2)
- added R15: 5.6k, open_bike_comp:1206_0603_hand_solder, B.Cu at (121.2, 93.0)
- added R16: 5.6k, open_bike_comp:1206_0603_hand_solder, B.Cu at (144.0, 85.5)
- added R17: 5.6k, open_bike_comp:1206_0603_hand_solder, B.Cu at (142.8, 81.0)
- added R18: 1k, open_bike_comp:1206_0603_hand_solder, B.Cu at (116.8, 93.0)
- added R19: 1k, open_bike_comp:1206_0603_hand_solder, B.Cu at (142.5, 77.5)
- added R2: 100k, open_bike_comp:1206_0603_hand_solder, B.Cu at (140.2, 130.0)
- added R20: 1k, open_bike_comp:1206_0603_hand_solder, B.Cu at (144.0, 92.2)
- added R21: 1k, open_bike_comp:1206_0603_hand_solder, B.Cu at (144.0, 90.0)
- added R22: 1k, open_bike_comp:1206_0603_hand_solder, B.Cu at (144.0, 83.2)
- added R23: 1k, open_bike_comp:1206_0603_hand_solder, B.Cu at (144.0, 87.8)
- added R24: 1k, open_bike_comp:1206_0603_hand_solder, B.Cu at (119.0, 93.0)
- added R27: 100k, open_bike_comp:1206_0603_hand_solder, B.Cu at (156.1, 113.0)
- added R3: 5.1k, open_bike_comp:1206_0603_hand_solder, B.Cu at (96.8, 137.1)
- added R4: 5.1k, open_bike_comp:1206_0603_hand_solder, B.Cu at (65.2, 136.9)
- added R5: 100k, open_bike_comp:1206_0603_hand_solder, B.Cu at (144.0, 126.5)
- added R6: 800k, open_bike_comp:1206_0603_hand_solder, B.Cu at (118.0, 87.0)
- added R7: 2M, open_bike_comp:1206_0603_hand_solder, B.Cu at (118.0, 89.2)
- added R8: 0, open_bike_comp:1206_0603_hand_solder, B.Cu at (175.4, 117.4)
- added R9: 0, open_bike_comp:1206_0603_hand_solder, B.Cu at (173.2, 117.4)
- added SW1: BATT_ON_OFF_SWITCH, nrfmicro:switch_MSK-12C02_smd, B.Cu at (116.5, 128.5)
- added SW2: SW_Push, open_bike_comp:KSC521JROHS_with_pad, F.Cu at (58.2, 139.9)
- added SW3: SW_Push, open_bike_comp:KSC521JROHS_with_pad, F.Cu at (87.6, 140.0)
- added SW4: SW_Push, open_bike_comp:KSC521JROHS_with_pad, F.Cu at (68.6, 140.0)
- added SW5: SW_Push, open_bike_comp:KSC521JROHS_with_pad, F.Cu at (97.7, 140.0)
- added U1: MCP73831-2-OT, Package_TO_SOT_SMD:SOT-23-5, B.Cu at (128.5, 129.0)
- added U10: LS027B7DH01, Connector_FFC-FPC:TE_1-1734839-0_1x10-1MP_P0.5mm_Horizontal, B.Cu at (154.2, 103.2)
- added U11: B39162B3913U410, open_bike_comp:B39162B3913U410, B.Cu at (138.5, 74.0)
- added U2: BME280, open_bike_comp:BME280, B.Cu at (164.8, 134.2)
- added U3: AP2112K-3.3, Package_TO_SOT_SMD:SOT-23-5, B.Cu at (143.8, 130.2)
- added U6: E73-2G4M08S1C-52840, nrfmicro:E73-2G4M08S1C-52840, B.Cu at (133.5, 117.0)
- added U9: SIM868, SIM868:XCVR_SIM868, B.Cu at (131.2, 85.5)
- added USB1: HRO-TYPE-C-31-M-12, nrfmicro:HRO-TYPE-C-31-M-12, B.Cu at (81.0, 148.5)
- added Y1: 32.768 kHz, Crystal:Crystal_DS26_D2.0mm_L6.0mm_Horizontal, B.Cu at (136.2, 111.2)
- added Z1: MMSZ5231BT1G, SamacSys_Parts:SOD3716X135N, B.Cu at (118.2, 84.2)
Routing:
- net Net-(C7-Pad1): track 0.00 -> 0.74 mm
- net GSM_RTS_UNREG: track 0.00 -> 0.55 mm
Other:
- board outline added: 109.5 x 85.6 mm
- board text added: "Active area"
- board text added: "Bottom plate is a 1mm offset of 3d case interior."
- board text added: "Centre of lcd"
- board text added: "PINOUT OF SIM IS WRONG"
- board text added: "SHOULD EXTRA PINS BE GROUNDED?"
- board text added: "SOLDER BRIDGE HERE ALSO"
- board text added: "This is the 3D case interior outline"
