File: pcb/bike_computer.sch (KiCad schematic (older format))
At the start: 44 parts

Commit message: Working on schematic
Parts:
- added C6, C9: 10uF, symbol Device:C
- added C7, C8: 1uF, symbol Device:C
- added J3: GND_pads, symbol Connector:Conn_01x05_Female
- added JP1: AD0_jumper, symbol Jumper:SolderJumper_3_Open
- added JP2: SWD_VCC, symbol Jumper:SolderJumper_3_Open
- added U5: MAX619, symbol open_bike_comp:MAX619
- J1: renamed from J?; value WirelessChargeConnn -> WirelessChargeConn
- J4: renamed from J?; value SWD Header -> SWD_header
- JP3: renamed from JP?; symbol Jumper:Jumper_3_Open -> Jumper:SolderJumper_3_Open
- U7: renamed from U?; footprint (none) -> open_bike_comp:BMP280
- gave numbers to parts that had none: 40
Connections:
- net labels added: 5V_SHDN, SIM_DTR, SIM_MIC+, SIM_MIC-, SIM_RING, VUSB
- net labels removed: 9AXIS_AD0, SMS_DTR, SMS_MIC+, SMS_MIC-
- wire segments 242 -> 305
- no-connect marks 11 -> 12
Other:
- note added: "5V boost"
- note added: "5V_SHDN should be pulled low for normal operation."
- note added: "Accelerometer, gyro and\nmagnetometer."
- note added: "Buttons"
- note added: "Chargeable by either USB or Qi. USB is preffered."
- note added: "If the capacitive sensors don't work, the \nground pads will make it easier to turn into \nbuttons"
- note added: "LCD and SD card each have their own SPI bus. Sensors share the I2C bus."
- note added: "Memory LCD's don't generate the VCOM signal required to \nprevent DC bias from building up. EXTCOMIN does this."
- note added: "Open source bike computer v1.0"
- note added: "SIM800L breakout module"
- note added: "Temperature and pressure sensor breakout"
- note added: "The voltage and high current requirements means powering directly \nfrom battery (>1.2Ah) is best. SIM800L has a battery indicator function.\nDTR is for sleep mode."
- note added: "https://github.com/HalFrgrd/Open-source-bike-computer"
- note removed: "Memory LCD's don't generate\nthe VCOM signal required to \nprevent DC bias from building up."
- note removed: "SIM"
- note removed: "Temperature and pressure sensor"
- note removed: "The voltage and high current requirements means powering directly \nfrom battery (>1.2Ah) is best"
- moved on the sheet: C1, C13, C14, C5, D2, H1, H2, H3, H4, H5, J2, J4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

Commit message: worked on schematic
Parts:
- removed U9: Micro_SD_Card_Module, symbol open_bike_comp:Micro_SD_Card_Module
- added AE1: Molex 204286-0001, symbol Device:Antenna
- added ANT1: ANT-LTE-SP610-T, SamacSys_Parts:ANTLTESP610T, symbol SamacSys_Parts:ANT-LTE-SP610-T
- added ANT2: SR4G053, SamacSys_Parts:SR4G053, symbol SamacSys_Parts:SR4G053
- added C15, C16, C17: 22pF, Capacitor_SMD:C_1206_3216Metric_Pad1.42x1.75mm_HandSolder, symbol Device:C
- added C18, C20: 0.1uF, Capacitor_SMD:C_1206_3216Metric_Pad1.42x1.75mm_HandSolder, symbol Device:C
- added C19: 10uF, Capacitor_SMD:C_1206_3216Metric_Pad1.42x1.75mm_HandSolder, symbol Device:C
- added C21: CP 100uF, symbol Device:CP
- added C22: 1uF, Capacitor_SMD:C_1206_3216Metric_Pad1.42x1.75mm_HandSolder, symbol Device:C
- added C23: 33pF, Capacitor_SMD:C_1206_3216Metric_Pad1.42x1.75mm_HandSolder, symbol Device:C
- added C24: 10pF, Capacitor_SMD:C_1206_3216Metric_Pad1.42x1.75mm_HandSolder, symbol Device:C
- added C25, C26: C, symbol Device:C
- added C27, C28: -, symbol Device:C
- added D3: ESDA6V1, SamacSys_Parts:SOT95P280X145-6N, symbol Power_Protection:SP0504BAJT
- added D4: 5.1V 500mW, symbol Device:D_Zener
- added D5: D_TVS, symbol Device:D_TVS
- added H6, H7, H8, H9: Mnt_Hole, MountingHole:MountingHole_3.2mm_M3_Pad_Via, symbol Mechanical:MountingHole_Pad
- added J6: SIM_Card, SamacSys_Parts:78646-3001, symbol Connector:SIM_Card
- added J7: Micro_SD_Card, symbol Connector:Micro_SD_Card
- added R12, R13, R14: 22R, symbol Device:R
- added R15, R16, R17: 5.6k, symbol Device:R
- added R18, R19, R20, R21, R22, R23, R24: 1k, symbol Device:R
- added R25, R26: 0, symbol Device:R
- added U11: B39162B3913U410, open_bike_comp:B39162B3913U410, symbol open_bike_comp:B39162B3913U410
- added U12: SKY65404, RF:Skyworks_SKY65404-31, symbol RF_Amplifier:SKY65404
- added U9: SIM868, SIM868:XCVR_SIM868, symbol SIM868:SIM868
- C1, C10, C11, C12, C13, C14, C2, C3, C4, C5, C6, C7, C8, C9: footprint (none) -> Capacitor_SMD:C_1206_3216Metric_Pad1.42x1.75mm_HandSolder
- D2: footprint (none) -> Diode_SMD:D_SOD-123
- J3: footprint (none) -> Connector_PinHeader_2.54mm:PinHeader_1x05_P2.54mm_Vertical
- J4: footprint (none) -> Connector_PinHeader_2.54mm:PinHeader_1x04_P2.54mm_Vertical
- JP3: footprint (none) -> Jumper:SolderJumper-3_P1.3mm_Open_RoundedPad1.0x1.5mm
- U10: footprint (none) -> Connector_FFC-FPC:TE_1-1734839-0_1x10-1MP_P0.5mm_Horizontal
- U4: footprint (none) -> open_bike_comp:GY-9250
- U6: footprint (none) -> nrfmicro:E73-2G4M08S1C-52840
- USB1: footprint (none) -> nrfmicro:HRO-TYPE-C-31-M-12
Connections:
- net labels added: 4V, 868_GPIO_1, 868_GPS_EN, 868_GPS_RXD, 868_GPS_TXD, 868_GSM_CTS, 868_GSM_RI, 868_GSM_RTS, 868_GSM_RXD, 868_GSM_TXD, 868_MICN, 868_MICP, 868_PWR, 868_RF_SYNC, 868_STATUS, GPS_ANT, GPS_RXD_UNREG, GPS_TXD_UNREG, GSM_ANT, GSM_CTS_UNREG, GSM_RI_UNREG, GSM_RTS_UNREG, GSM_RXD_UNREG, GSM_TXD_UNREG, POSSIBLY4V, SIM_CLK, SIM_DATA, SIM_VCC
- net labels removed: SMS_RING
- wire segments 305 -> 440
- no-connect marks 12 -> 55
Other:
- note added: "Check power supply for SIM card."
- note added: "Keeping VRTC powered helps to decrease cold start time."
- note added: "Logic level shift"
- note added: "Must generate clock signal."
- note added: "Possibly use 1pps\n"
- note added: "SD card"
- note added: "SIM868 UART uses 3.0V max, so we shift down \n3.3V to (5.6-1)/5.6 * 3.3 = 2.7."
- note added: "SIM868e (SIM + GPS)"
- moved on the sheet: C10, C11, C12, C13, C14, C6, C7, C8, C9, H1, H2, H3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

Commit message: Assigning footprints
Parts:
- removed J7: Micro_SD_Card, symbol Connector:Micro_SD_Card
- added J10: Cap_button_5_conn, Connector_PinHeader_2.54mm:PinHeader_1x01_P2.54mm_Vertical, symbol Connector:Conn_01x01_Female
- added J11: 47219-2001, SamacSys_Parts:472192001, symbol SamacSys_Parts:47219-2001
- added J5: Cap_button_1_conn, Connector_PinHeader_2.54mm:PinHeader_1x01_P2.54mm_Vertical, symbol Connector:Conn_01x01_Female
- added J7: Cap_button_2_conn, Connector_PinHeader_2.54mm:PinHeader_1x01_P2.54mm_Vertical, symbol Connector:Conn_01x01_Female
- added J8: Cap_button_3_conn, Connector_PinHeader_2.54mm:PinHeader_1x01_P2.54mm_Vertical, symbol Connector:Conn_01x01_Female
- added J9: Cap_button_4_conn, Connector_PinHeader_2.54mm:PinHeader_1x01_P2.54mm_Vertical, symbol Connector:Conn_01x01_Female
- C1, C10, C11, C12, C13, C14, C15, C16, C17, C18, C19, C2, C20, C22, C23, C24, C3, C4, C5, C6, C7, C8, C9: footprint Capacitor_SMD:C_1206_3216Metric_Pad1.42x1.75mm_HandSolder -> open_bike_comp:1206_0603_hand_solder
- H1, H2, H3, H4, H5: footprint (none) -> open_bike_comp:touch_pad_1
- J1: footprint (none) -> Connector_PinHeader_2.54mm:PinHeader_1x02_P2.54mm_Vertical
- J2: footprint (none) -> Connector_JST:JST_PH_S2B-PH-K_1x02_P2.00mm_Horizontal
- JP1, JP2: footprint (none) -> Jumper:SolderJumper-3_P1.3mm_Open_RoundedPad1.0x1.5mm
- R1, R10, R11, R12, R13, R14, R15, R16, R17, R18, R19, R2, R20, R21, R22, R23, R24, R3, R4, R5, R6, R7, R8, R9: footprint (none) -> open_bike_comp:1206_0603_hand_solder
- Y1: footprint (none) -> Crystal:Crystal_DS26_D2.0mm_L6.0mm_Horizontal
Connections:
- net 5V_SHDN: no longer U6.26 (P0.18/RESET)
- net CAP_BUTTON_1: now also J5.1 (Pin_1); no longer H1.1
- net CAP_BUTTON_2: now also J7.1 (Pin_1); no longer H2.1
- net CAP_BUTTON_3: now also J8.1 (Pin_1); no longer H3.1
- net CAP_BUTTON_4: now also J9.1 (Pin_1); no longer H4.1
- net CAP_BUTTON_5: now also J10.1 (Pin_1); no longer H5.1
- net GND: now also J11.10 (GND_2), J11.11 (GND_3), J11.12 (GND_4), J11.6 (VSS), J11.9 (GND_1)
- net LCD_DISP: now also U6.26 (P0.18/RESET)
- net SC_CARD_MISO: now also J11.7 (DAT0)
- net SD_CARD_CLK: now also J11.5 (CLK)
- net SD_CARD_CS: now also J11.2 (CD/DAT3)
- net SD_CARD_MOSI: now also J11.3 (CMD)
- net VCC: now also J11.4 (VDD)
- no-connect marks 55 -> 54
Other:
- note added: "No need for card insertion detection; card is always in."
- note added: "PULL LOW"
- note removed: "For cost and convenience purposes, I'm using a breakout.\nNo need for card insertion detection; card is always in."
- moved on the sheet: H1, H2, H3, H4, H5, J3

Commit message: Sorting out 2 plate design
Parts:
- removed AE1: Molex 204286-0001, symbol Device:Antenna
- removed ANT1: ANT-LTE-SP610-T, SamacSys_Parts:ANTLTESP610T, symbol SamacSys_Parts:ANT-LTE-SP610-T
- removed ANT2: SR4G053, SamacSys_Parts:SR4G053, symbol SamacSys_Parts:SR4G053
- removed C13: 0.1uF, open_bike_comp:1206_0603_hand_solder, symbol Device:C
- removed C14, C9: 10uF, open_bike_comp:1206_0603_hand_solder, symbol Device:C
- removed C21: CP 100uF, symbol Device:CP
- removed D1: D, symbol Device:D
- removed D4: 5.1V 500mW, symbol Device:D_Zener
- removed D5: D_TVS, symbol Device:D_TVS
- removed H7, H8, H9: Mnt_Hole, MountingHole:MountingHole_3.2mm_M3_Pad_Via, symbol Mechanical:MountingHole_Pad
- removed J3: GND_pads, Connector_PinHeader_2.54mm:PinHeader_1x05_P2.54mm_Vertical, symbol Connector:Conn_01x05_Female
- removed U12: SKY65404, RF:Skyworks_SKY65404-31, symbol RF_Amplifier:SKY65404
- removed U2: SIM800L_module, symbol open_bike_comp:SIM800L_module
- removed U5: MAX619, symbol open_bike_comp:MAX619
- removed U8: L96-M33, symbol open_bike_comp:L96-M33
- added ANT1: W3010, SamacSys_Parts:ANTC10032X400N, symbol SamacSys_Parts:W3010
- added ANT2: W3073, SamacSys_Parts:ANTC10032X410N, symbol SamacSys_Parts:W3073
- added C9: TAJC107K006SNJ, SamacSys_Parts:CAPPM6032X280N, symbol SamacSys_Parts:TAJC107K006SNJ
- added D1, D4: 1N5819, Diode_SMD:D_SOD-123, symbol Device:D_Schottky
- added H? (x3): Mnt_Hole_1_Bot, MountingHole:MountingHole_3.2mm_M3_Pad_Via, symbol Mechanical:MountingHole_Pad
- added H? (x4): Mnt_Hole_1_Top, MountingHole:MountingHole_3.2mm_M3_Pad_Via, symbol Mechanical:MountingHole_Pad
- added IC1: REG71050DDCR, SamacSys_Parts:SOT95P280X110-6N, symbol SamacSys_Parts:REG71050DDCR
- added J12, J14: SAMTEC-FTSH-104-01-X-DV, open_bike_comp:SAMTEC-FTSH-104-01-X-DV, symbol open_bike_comp:SAMTEC-FTSH-104-01-X-DV
- added J13, J3: SAMTEC-CLP-104-02-X-D, open_bike_comp:SAMTEC-CLP-104-02-X-D, symbol open_bike_comp:SAMTEC-CLP-104-02-X-D
- added R27: 100k, open_bike_comp:1206_0603_hand_solder, symbol Device:R
- added SW1: SW_DPDT_x2, symbol Switch:SW_DPDT_x2
- added SW2, SW3, SW4, SW5, SW6: SW_Push, symbol Switch:SW_Push
- added Z1: MMSZ5231BT1G, SamacSys_Parts:SOD3716X135N, symbol SamacSys_Parts:MMSZ5231BT1G
- C25, C26: value C -> NA; footprint (none) -> open_bike_comp:1206_0603_hand_solder
- C27, C28, R25, R26: footprint (none) -> open_bike_comp:1206_0603_hand_solder
- C6: value 10uF -> 1uF
- C7: value 1uF -> 0.1uF
- C8: value 1uF -> 10uF
- H6: value Mnt_Hole -> Mnt_Hole_1_Bot
Connections:
- net 4V is gone; now on net VCC: C19.1, C20.1, U9.34 (GPS_VBAT)
- net NFC1 is gone; now on net 868_RF_SYNC: U6.41 (P0.09/NFC1)
- net NFC2 is gone; now on net 868_GPS_EN: U6.43 (P0.10/NFC2)
- net 5V: now also C8.1, IC1.1 (VOUT)
- net BATT_V_IND: now also U9.38 (ADC); no longer U6.18 (P0.04/AIN2)
- net CAP_BUTTON_1: now also J13.1, J14.1
- net CAP_BUTTON_2: now also J13.3, J14.3
- net CAP_BUTTON_3: now also J13.5, J14.5
- net CAP_BUTTON_4: now also J13.7, J14.7
- net CAP_BUTTON_5: now also J13.2, J14.2
- net CHARG_STAT: now also U9.57 (GPIO1)
- net GND: now also C8.2, C9.2, H?.1, H?.1, H?.1, H?.1, H?.1, H?.1, H?.1, IC1.2 (GND), J12.1, J13.4, J14.4, J3.1, Z1.2
- net VBATT: now also C9.1, J12.3, J12.4, J3.3, J3.4, SW1.2 (B), Z1.1; no longer Q1.3 (D), R6.1
- net VBUS: now also D1.2 (A)
- net VCC: now also J12.2, J3.2, R27.1; no longer C6.1
- net at U1.4 (VDD): now also D1.1 (K), D4.1 (K); no longer J1.1 (Pin_1)
- net VIN: now reaches C1.1, D2.1 (K), Q1.2 (S), R5.1, U3.1 (VIN)
- net VIN: now also C6.1, IC1.5 (VIN)
- net at C7.1: now also IC1.6 (C_PUMP+)
- net at C7.2: now also IC1.4 (CPUMP-)
- net at C26.1, R25.1: now also ANT2.1 (FEED)
- net at C27.1, R26.2: now also U11.2 (INPUT)
- net at C28.1, R26.1: now also ANT1.1 (FEED)
- new net: Q1.3 (D), R6.1, SW1.1 (A)
- new net: D4.2 (A), J1.1 (Pin_1)
- new net: IC1.3 (ENABLE), R27.2
- no-connect marks 54 -> 41
Other:
- note added: "2.9V to 4.4V"
- note added: "Bottom connectors"
- note added: "Bottom plate holes"
- note added: "Chargeable by either USB or Qi."
- note added: "Connectors between the two PCBs"
- note added: "Mounting holes"
- note added: "Plan for FLEx display"
- note added: "RECHECK POWER SUPPLY"
- note added: "SIM868 has a built in LNA, but it does recommend using a SAW filter.\n"
- note added: "The reference design doesn't use ESD protection here, seems optional. \nSo I'm not using it either."
- note added: "Top connectors"
- note added: "Top plate holes"
- note removed: "5V_SHDN should be pulled low for normal operation."
- note removed: "Chargeable by either USB or Qi. USB is preffered."
- note removed: "GPS"
- note removed: "PULL LOW"
- note removed: "SIM800L breakout module"
- note removed: "The voltage and high current requirements means powering directly \nfrom battery (>1.2Ah) is best. SIM800L has a battery indicator function.\nDTR is for sleep mode."
- moved on the sheet: C23, C24, C25, C26, C27, C28, H6, J1, R25, R26, R3, R4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

Commit message: Sorted main layout
Parts:
- removed ANT1: W3010, SamacSys_Parts:ANTC10032X400N, symbol SamacSys_Parts:W3010
- removed ANT2: W3073, SamacSys_Parts:ANTC10032X410N, symbol SamacSys_Parts:W3073
- removed C25, C26: NA, open_bike_comp:1206_0603_hand_solder, symbol Device:C
- removed C27, C28: -, open_bike_comp:1206_0603_hand_solder, symbol Device:C
- removed H1: Capacitive_button_1, open_bike_comp:touch_pad_1, symbol Mechanical:MountingHole_Pad
- removed H2: Capacitive_button_2, open_bike_comp:touch_pad_1, symbol Mechanical:MountingHole_Pad
- removed H3: Capacitive_button_3, open_bike_comp:touch_pad_1, symbol Mechanical:MountingHole_Pad
- removed H4: Capacitive_button_4, open_bike_comp:touch_pad_1, symbol Mechanical:MountingHole_Pad
- removed H5: Capacitive_button_5, open_bike_comp:touch_pad_1, symbol Mechanical:MountingHole_Pad
- removed H6, H? (x3): Mnt_Hole_1_Bot, MountingHole:MountingHole_3.2mm_M3_Pad_Via, symbol Mechanical:MountingHole_Pad
- removed J10: Cap_button_5_conn, Connector_PinHeader_2.54mm:PinHeader_1x01_P2.54mm_Vertical, symbol Connector:Conn_01x01_Female
- removed J12, J14: SAMTEC-FTSH-104-01-X-DV, open_bike_comp:SAMTEC-FTSH-104-01-X-DV, symbol open_bike_comp:SAMTEC-FTSH-104-01-X-DV
- removed J13, J3: SAMTEC-CLP-104-02-X-D, open_bike_comp:SAMTEC-CLP-104-02-X-D, symbol open_bike_comp:SAMTEC-CLP-104-02-X-D
- removed J5: Cap_button_1_conn, Connector_PinHeader_2.54mm:PinHeader_1x01_P2.54mm_Vertical, symbol Connector:Conn_01x01_Female
- removed J6: SIM_Card, SamacSys_Parts:78646-3001, symbol Connector:SIM_Card
- removed J7: Cap_button_2_conn, Connector_PinHeader_2.54mm:PinHeader_1x01_P2.54mm_Vertical, symbol Connector:Conn_01x01_Female
- removed J8: Cap_button_3_conn, Connector_PinHeader_2.54mm:PinHeader_1x01_P2.54mm_Vertical, symbol Connector:Conn_01x01_Female
- removed J9: Cap_button_4_conn, Connector_PinHeader_2.54mm:PinHeader_1x01_P2.54mm_Vertical, symbol Connector:Conn_01x01_Female
- removed JP2: SWD_VCC, Jumper:SolderJumper-3_P1.3mm_Open_RoundedPad1.0x1.5mm, symbol Jumper:SolderJumper_3_Open
- removed R25, R26: 0, open_bike_comp:1206_0603_hand_solder, symbol Device:R
- removed SW6: SW_Push, symbol Switch:SW_Push
- removed U4: MPU_9250, open_bike_comp:GY-9250, symbol open_bike_comp:MPU_9250
- removed U7: BMP280, open_bike_comp:BMP280, symbol open_bike_comp:BMP280
- added ANT1: SR4G008, SR4G008, symbol SamacSys_Parts:SR4G008
- added ANT2: CONUFL001-SMD, CONUFL001-SMD, symbol SamacSys_Parts:CONUFL001-SMD
- added C13, C14, C21: 0.1uF, open_bike_comp:1206_0603_hand_solder, symbol Device:C
- added IC2: MPU-9250, SamacSys_Parts:QFN40P300X300X105-25N-D, symbol SamacSys_Parts:MPU-9250
- added J3: Conn_01x10_TopPlate, open_bike_comp:10_smd_connector, symbol Connector_Generic_MountingPin:Conn_01x10_MountingPin
- added J5: Conn_01x10_BotPlate, Connector_PinHeader_2.54mm:PinHeader_1x10_P2.54mm_Vertical, symbol Connector_Generic_MountingPin:Conn_01x10_MountingPin
- added J6: 78646-3001, 78646-3001, symbol SamacSys_Parts:78646-3001
- added U2: BME280, open_bike_comp:BME280, symbol open_bike_comp:BME280
- H11: renamed from H?; value Mnt_Hole_1_Top -> Mnt_Hole_3_Top; footprint MountingHole:MountingHole_3.2mm_M3_Pad_Via -> open_bike_comp:R303000402; symbol Mechanical:MountingHole_Pad -> Mechanical:MountingHole
- H13: renamed from H?; value Mnt_Hole_1_Top -> Mnt_Hole_4_Top; footprint MountingHole:MountingHole_3.2mm_M3_Pad_Via -> open_bike_comp:R303000402; symbol Mechanical:MountingHole_Pad -> Mechanical:MountingHole
- H7: renamed from H?; footprint MountingHole:MountingHole_3.2mm_M3_Pad_Via -> open_bike_comp:R303000402; symbol Mechanical:MountingHole_Pad -> Mechanical:MountingHole
- H9: renamed from H?; value Mnt_Hole_1_Top -> Mnt_Hole_2_Top; footprint MountingHole:MountingHole_3.2mm_M3_Pad_Via -> open_bike_comp:R303000402; symbol Mechanical:MountingHole_Pad -> Mechanical:MountingHole
- J1: footprint Connector_PinHeader_2.54mm:PinHeader_1x02_P2.54mm_Vertical -> Connector_PinHeader_1.27mm:PinHeader_1x02_P1.27mm_Vertical
- J2: footprint Connector_JST:JST_PH_S2B-PH-K_1x02_P2.00mm_Horizontal -> Connector_PinHeader_1.27mm:PinHeader_1x02_P1.27mm_Vertical
- SW1: value SW_DPDT_x2 -> BATT_ON_OFF_SWITCH; footprint (none) -> nrfmicro:switch_MSK-12C02_smd; symbol Switch:SW_DPDT_x2 -> Switch:SW_DPST_x2
- SW2, SW3, SW4, SW5: footprint (none) -> open_bike_comp:KSC521JROHS_with_pad
Connections:
- net CAP_BUTTON_5 is gone; now on net 868_PWR: U6.15 (P0.05/AIN3)
- net 9AXIS_INT: now also IC2.12 (INT)
- net 9AXIS_SCL: now also IC2.23 (SCL/SCLK), U2.3 (SCL)
- net 9AXIS_SDA: now also IC2.24 (SDA/SDI), U2.4 (SDA)
- net CAP_BUTTON_1: now also SW2.1, J3.1 (Pin_1), J5.1 (Pin_1)
- net CAP_BUTTON_2: now also SW3.1, J3.2 (Pin_2), J5.2 (Pin_2)
- net CAP_BUTTON_3: now also SW4.1, J3.9 (Pin_9), J5.9 (Pin_9)
- net CAP_BUTTON_4: now also SW5.1, J3.10 (Pin_10), J5.10 (Pin_10)
- net GND: now also ANT1.3 (GND_1), ANT1.4 (GND_2), ANT1.6 (GND_3), ANT2.2 (GND_1), ANT2.3 (GND_2), C13.2, C14.1, C21.2, IC2.11 (FSYNC), IC2.18 (GND), IC2.20 (RESV_3), J3.7 (Pin_7), J5.7 (Pin_7), J6.4 (C5), U2.2 (GND); no longer H11.1, H13.1, H7.1, H9.1
- net GSM_ANT: now also ANT2.1 (SIG)
- net SIM_VCC: now also J6.1 (C1)
- net USB_D+: now also J3.5 (Pin_5), J5.5 (Pin_5)
- net USB_D-: now also J3.6 (Pin_6), J5.6 (Pin_6)
- net VBATT: now also SW1.1 (A); no longer SW1.2 (B)
- net VBUS: now also J4.1 (Pin_1), J3.3 (Pin_3), J5.3 (Pin_3)
- net VCC: now also SW2.2, SW3.2, SW4.2, SW5.2, C13.1, C21.1, IC2.1 (RESV_1), IC2.13 (VDD), IC2.22 (~CS), IC2.8 (VDDIO), J3.4 (Pin_4), J5.4 (Pin_4), U2.1 (VIN)
- net at Q1.3 (D), R6.1: now also SW1.2 (B); no longer SW1.1 (A)
- net at JP1.1 (A): now also IC2.9 (AD0/SDO)
- net at D3.3 (K), R14.1: now also J6.2 (C2)
- net at D3.4 (K), R13.1: now also J6.3 (C3)
- net at D3.5 (K), R12.1: now also J6.6 (C7)
- net at U11.2 (INPUT): now also ANT1.2 (FEED)
- new net: C14.2, IC2.10 (REGOUT)
- no-connect marks 41 -> 53
Other:
- note added: "Accelerometer, gyro and magnetometer.\nMPU-9250 is outdated but it runs at 3.3v unlike ICM20948"
- note added: "BME280 breakout\n"
- note added: "Bottom plate"
- note added: "R30-3000402"
- note added: "Temperature, pressure, humidity sensor breakout"
- note added: "Top plate"
- note removed: "Accelerometer, gyro and\nmagnetometer."
- note removed: "Bottom connectors"
- note removed: "Bottom plate holes"
- note removed: "No humidity for the BMP280 (only BME280).\n"
- note removed: "Temperature and pressure sensor breakout"
- note removed: "Top connectors"
- moved on the sheet: JP1, SW2, SW3, SW4, SW5
